File: hardware/ntp_7seg_clock.sch (KiCad schematic (older format))
At the start: 42 parts, among them J1 Barrel_Jack, J2 Conn_02x04_Odd_Even, J3 Conn_02x04_Odd_Even, J4 Conn_02x04_Odd_Even, J5 Conn_02x04_Odd_Even, J6 Conn_01x06_Male, Q1 NJL7302L-F3, Q2 Q_NPN_BEC, Q3 Q_NPN_BEC, SW1 SW_PUSH_SMALL_H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

Commit message: Improved RTC 3V3 backup voltage handling
Parts:
- removed D3: SBD 40V 200mA, Diodes_SMD:D_0603, symbol device:D_Zener_Small
- added C12: 2.2u, Capacitor_SMD:C_0603_1608Metric, symbol ntp_7seg_clock-rescue:C-device
- added C13: 10u/35V, Capacitor_SMD:C_0805_2012Metric, symbol ntp_7seg_clock-rescue:C_Small-device
- added D3, D4, D5: ESD5Z3.3T1G, Diode_SMD:D_SOD-323_HandSoldering, symbol ntp_7seg_clock-rescue:D_Zener_Small-device
- added D6, D7: 1N4148W, Diode_SMD:D_SOD-323, symbol Diode:1N4148W
- added J7: USB_B_Micro, components:USB_Micro-B_Jing_A01SB141B1-067, symbol Connector:USB_B_Micro
- added Q4: AO3401, Package_TO_SOT_SMD:SOT-23, symbol Device:Q_NMOS_GSD
- added R12: 1M, Resistor_SMD:R_0603_1608Metric, symbol ntp_7seg_clock-rescue:R-device
- added R13: 22K, Resistor_SMD:R_0603_1608Metric, symbol ntp_7seg_clock-rescue:R-device
- added R14: 120R, Resistor_SMD:R_0603_1608Metric, symbol ntp_7seg_clock-rescue:R-device
- added U6: SE8533X2-HF, Package_TO_SOT_SMD:SOT-23, symbol Regulator_Linear:MCP1703A-3302_SOT23
- C1, C11, C2, C3, C4, C5, C6, C7, C9: symbol device:C_Small -> ntp_7seg_clock-rescue:C_Small-device
- C10: symbol device:C -> ntp_7seg_clock-rescue:C-device
- C8: symbol device:CP1_Small -> ntp_7seg_clock-rescue:CP1_Small-device
- D1: value D_Zener_Small -> 28V TVS; footprint Diodes_SMD:D_SOD-123F -> Diode_SMD:D_SMA; symbol device:D_Zener_Small -> Device:D_TVS
- D2: symbol device:LED -> ntp_7seg_clock-rescue:LED-device
- F1: value Polyfuse_Small -> 1A hold; footprint Capacitors_SMD:C_1812_HandSoldering -> Fuse:Fuse_1812_4532Metric; symbol device:Polyfuse_Small -> ntp_7seg_clock-rescue:Polyfuse_Small-device
- J1: symbol Connector:Barrel_Jack -> ntp_7seg_clock-rescue:Barrel_Jack-Connector
- J2, J3, J4, J5: symbol Connector:Conn_02x04_Odd_Even -> ntp_7seg_clock-rescue:Conn_02x04_Odd_Even-Connector
- L1: symbol device:L_Small -> ntp_7seg_clock-rescue:L_Small-device
- Q2, Q3: symbol device:Q_NPN_BEC -> ntp_7seg_clock-rescue:Q_NPN_BEC-device
- R1, R10, R11, R2, R3, R5, R6, R7, R8, R9: symbol device:R -> ntp_7seg_clock-rescue:R-device
- R4: value 10R -> 1k; symbol device:R -> ntp_7seg_clock-rescue:R-device
- U4: symbol philips:PCF8563 -> ntp_7seg_clock-rescue:PCF8563-philips
Connections:
- net labels added: 3V3+, 3V3_RTC
- wire segments 160 -> 194
Other:
- note added: "3.3V + Vf(D6)"
- note added: "As close \nas possible"
- note added: "ESD diode abused as zener"

Commit message: Ooops reverse protection FET is reversed; and others
Parts:
- removed D5: ESD5Z3.3T1G, Diode_SMD:D_SOD-323_HandSoldering, symbol ntp_7seg_clock-rescue:D_Zener_Small-device
- C8: value EDLC -> ML621; footprint components:BAT_6814_LAY -> components:BAT_MS621T_LAY; symbol ntp_7seg_clock-rescue:CP1_Small-device -> Device:Battery_Cell
Other:
- moved on the sheet: D3, R12, R13
Changed lines of the file:
@@
 $EndComp
 $Comp
-L ntp_7seg_clock-rescue:CP1_Small-device C8
+L Device:Battery_Cell C8
 U 1 1 5BE90BEB
-P 8000 9850
-F 0 "C8" H 8091 9896 50  0000 L CNN
-F 1 "EDLC" H 8091 9805 50  0000 L CNN
-F 2 "components:BAT_6814_LAY" H 8000 9850 50  0001 C CNN
-F 3 "" H 8000 9850 50  0001 C CNN
-	1    8000 9850
+P 8000 9950
+F 0 "C8" H 8091 9996 50  0000 L CNN
+F 1 "ML621" H 8091 9905 50  0000 L CNN
+F 2 "components:BAT_MS621T_LAY" H 8000 9950 50  0001 C CNN
+F 3 "" H 8000 9950 50  0001 C CNN
+	1    8000 9950
 	1    0    0    -1
 $EndComp
@@
 Wire Wire Line
 	1150 1150 1250 1150
-Text Label 3200 1150 0    50   ~ 0
+Text Label 3900 1150 0    50   ~ 0
 VIN
 $Comp
@@
 L power:GND #PWR014
 U 1 1 5BFEB404
-P 8000 9950
-F 0 "#PWR014" H 8000 9700 50  0001 C CNN
-F 1 "GND" H 8005 9777 50  0000 C CNN
-F 2 "" H 8000 9950 50  0000 C CNN
-F 3 "" H 8000 9950 50  0000 C CNN
-	1    8000 9950
+P 8000 10050
+F 0 "#PWR014" H 8000 9800 50  0001 C CNN
+F 1 "GND" H 8005 9877 50  0000 C CNN
+F 2 "" H 8000 10050 50  0000 C CNN
+F 3 "" H 8000 10050 50  0000 C CNN
+	1    8000 10050
 	1    0    0    -1
 $EndComp
@@
 F 3 "~" H 2850 1250 50  0001 C CNN
 	1    2850 1250
-	0    -1   -1   0
+	0    1    -1   0
 $EndComp
 $Comp
 L ntp_7seg_clock-rescue:R-device R12
 U 1 1 5BED39AE
-P 2350 1550
-F 0 "R12" H 2420 1596 50  0000 L CNN
-F 1 "1M" H 2420 1505 50  0000 L CNN
-F 2 "Resistor_SMD:R_0603_1608Metric" V 2280 1550 50  0001 C CNN
-F 3 "" H 2350 1550 50  0001 C CNN
-	1    2350 1550
+P 3150 1450
+F 0 "R12" H 3220 1496 50  0000 L CNN
+F 1 "1M" H 3220 1405 50  0000 L CNN
+F 2 "Resistor_SMD:R_0603_1608Metric" V 3080 1450 50  0001 C CNN
+F 3 "" H 3150 1450 50  0001 C CNN
+	1    3150 1450
 	1    0    0    1
 $EndComp
@@
 L ntp_7seg_clock-rescue:R-device R13
 U 1 1 5BED414D
-P 2350 1900
-F 0 "R13" H 2420 1946 50  0000 L CNN
-F 1 "22K" H 2420 1855 50  0000 L CNN
-F 2 "Resistor_SMD:R_0603_1608Metric" V 2280 1900 50  0001 C CNN
-F 3 "" H 2350 1900 50  0001 C CNN
-	1    2350 1900
+P 3150 1850
+F 0 "R13" H 3220 1896 50  0000 L CNN
+F 1 "22K" H 3220 1805 50  0000 L CNN
+F 2 "Resistor_SMD:R_0603_1608Metric" V 3080 1850 50  0001 C CNN
+F 3 "" H 3150 1850 50  0001 C CNN
+	1    3150 1850
 	1    0    0    1
 $EndComp
-Wire Wire Line
-	2350 1700 2350 1750
-Connection ~ 2650 1150
 $Comp
 L ntp_7seg_clock-rescue:D_Zener_Small-device D3
 U 1 1 5BEEF4FC
-P 2650 1500
-F 0 "D3" V 2604 1568 50  0000 L CNN
-F 1 "ESD5Z3.3T1G" V 2750 1550 50  0000 L CNN
-F 2 "Diode_SMD:D_SOD-323_HandSoldering" V 2650 1500 50  0001 C CNN
-F 3 "https://en.wikipedia.org/wiki/Zener_diode" V 2650 1500 50  0001 C CNN
-	1    2650 1500
+P 3450 1400
+F 0 "D3" V 3404 1468 50  0000 L CNN
+F 1 "ESD5Z3.3T1G" V 3550 1450 50  0000 L CNN
+F 2 "Diode_SMD:D_SOD-323_HandSoldering" V 3450 1400 50  0001 C CNN
+F 3 "https://en.wikipedia.org/wiki/Zener_diode" V 3450 1400 50  0001 C CNN
+	1    3450 1400
 	0    1    1    0
 $EndComp
-Wire Wire Line
-	2650 1600 2650 1750
-Wire Wire Line
-	2650 1750 2350 1750
-Connection ~ 2350 1750
-Wire Wire Line
-	2650 1750 2850 1750
-Wire Wire Line
-	2850 1750 2850 1450
-Connection ~ 2650 1750
 $Comp
 L power:GND #PWR030
 U 1 1 5BF0373E
-P 2350 2050
-F 0 "#PWR030" H 2350 1800 50  0001 C CNN
-F 1 "GND" H 2355 1877 50  0000 C CNN
-F 2 "" H 2350 2050 50  0001 C CNN
-F 3 "" H 2350 2050 50  0001 C CNN
-	1    2350 2050
+P 3150 2000
+F 0 "#PWR030" H 3150 1750 50  0001 C CNN
+F 1 "GND" H 3155 1827 50  0000 C CNN
+F 2 "" H 3150 2000 50  0001 C CNN
+F 3 "" H 3150 2000 50  0001 C CNN
+	1    3150 2000
 	1    0    0    -1
 $EndComp
@@
 	1600 1150 1950 1150
 Wire Wire Line
-	3200 1150 3050 1150
-Text Notes 2600 1850 0    50   ~ 0
+	3900 1150 3150 1150
+Text Notes 3100 2350 0    50   ~ 0
 ESD diode abused as zener
 Wire Wire Line
 	1250 1150 1600 1150
 Connection ~ 1250 1150
-Wire Wire Line
-	2150 1150 2350 1150
 $Comp
 L power:GND #PWR031
@@
 	1    0    0    -1
 $EndComp
-$Comp
-L ntp_7seg_clock-rescue:D_Zener_Small-device D5
-U 1 1 5BE9A523
-P 2650 1300
-F 0 "D5" V 2604 1368 50  0000 L CNN
-F 1 "ESD5Z3.3T1G" V 2750 1350 50  0000 L CNN
-F 2 "Diode_SMD:D_SOD-323_HandSoldering" V 2650 1300 50  0001 C CNN
-F 3 "https://en.wikipedia.org/wiki/Zener_diode" V 2650 1300 50  0001 C CNN
-	1    2650 1300
-	0    -1   -1   0
-$EndComp
-Wire Wire Line
-	2650 1200 2650 1150
-Wire Wire Line
-	2350 1400 2350 1150
-Connection ~ 2350 1150
-Wire Wire Line
-	2350 1150 2650 1150
 $Comp
 L Regulator_Linear:MCP1703A-3302_SOT23 U6
@@
 Text Notes 8200 8150 0    50   ~ 0
 3.3V + Vf(D6)
+Wire Wire Line
+	2150 1150 2650 1150
+Wire Wire Line
+	3150 1600 2850 1600
+Wire Wire Line
+	2850 1600 2850 1450
+Wire Wire Line
+	3150 1300 3150 1150
+Connection ~ 3150 1150
+Wire Wire Line
+	3150 1150 3050 1150
+Wire Wire Line
+	3450 1300 3150 1300
+Connection ~ 3150 1300
+Wire Wire Line
+	3450 1500 3450 1600
+Wire Wire Line
+	3450 1600 3150 1600
+Connection ~ 3150 1600
+Wire Wire Line
+	3150 1600 3150 1700
 $EndSCHEMATC

Commit message: Modified to use Li-ion rechargable battery
Parts:
- removed C13: 10u/35V, Capacitor_SMD:C_0805_2012Metric, symbol ntp_7seg_clock-rescue:C_Small-device
- removed D6: 1N4148W, Diode_SMD:D_SOD-323, symbol Diode:1N4148W
- removed U6: SE8533X2-HF, Package_TO_SOT_SMD:SOT-23, symbol Regulator_Linear:MCP1703A-3302_SOT23
- added Q5: Q_NPN_BEC, Package_TO_SOT_SMD:SOT-23, symbol ntp_7seg_clock-rescue:Q_NPN_BEC-device
- added Q6: AO3401, Package_TO_SOT_SMD:SOT-23, symbol Device:Q_NMOS_GSD
- added R15, R16: 10k, Resistor_SMD:R_0603_1608Metric, symbol ntp_7seg_clock-rescue:R-device
- D7: value 1N4148W -> SBD; symbol Diode:1N4148W -> Device:D_Schottky_Small
Connections:
- net labels removed: 3V3+
Other:
- note removed: "3.3V + Vf(D6)"
- note removed: "As close \nas possible"
Changed lines of the file:
@@
 Connection ~ 1250 1150
 $Comp
-L power:GND #PWR031
-U 1 1 5C0CA06C
-P 7650 9000
-F 0 "#PWR031" H 7650 8750 50  0001 C CNN
-F 1 "GND" H 7655 8827 50  0000 C CNN
-F 2 "" H 7650 9000 50  0000 C CNN
-F 3 "" H 7650 9000 50  0000 C CNN
-	1    7650 9000
-	1    0    0    -1
-$EndComp
-$Comp
-L Regulator_Linear:MCP1703A-3302_SOT23 U6
-U 1 1 5BEA2D6A
-P 7650 8250
-F 0 "U6" H 7650 8492 50  0000 C CNN
-F 1 "SE8533X2-HF" H 7650 8401 50  0000 C CNN
-F 2 "Package_TO_SOT_SMD:SOT-23" H 7650 8450 50  0001 C CNN
-F 3 "http://ww1.microchip.com/downloads/en/DeviceDoc/20005122B.pdf" H 7650 8200 50  0001 C CNN
-	1    7650 8250
-	1    0    0    -1
-$EndComp
-$Comp
-L Diode:1N4148W D6
-U 1 1 5BEAE0DE
-P 7650 8700
-F 0 "D6" V 7696 8620 50  0000 R CNN
-F 1 "1N4148W" V 7605 8620 50  0000 R CNN
-F 2 "Diode_SMD:D_SOD-323" H 7650 8525 50  0001 C CNN
-F 3 "https://www.vishay.com/docs/85748/1n4148w.pdf" H 7650 8700 50  0001 C CNN
-	1    7650 8700
+L Device:D_Schottky_Small D7
+U 1 1 5BF6DCC5
+P 8850 8750
+F 0 "D7" V 8896 8670 50  0000 R CNN
+F 1 "SBD" V 8805 8670 50  0000 R CNN
+F 2 "Diode_SMD:D_SOD-323" H 8850 8575 50  0001 C CNN
+F 3 "https://www.vishay.com/docs/85748/1n4148w.pdf" H 8850 8750 50  0001 C CNN
+	1    8850 8750
 	0    -1   -1   0
 $EndComp
-Text Label 7150 8250 0    50   ~ 0
-VIN
-Wire Wire Line
-	7350 8250 7150 8250
-$Comp
-L ntp_7seg_clock-rescue:C_Small-device C13
-U 1 1 5BEEDD3E
-P 8200 8500
-F 0 "C13" V 8000 8450 50  0000 L CNN
-F 1 "10u/35V" V 8100 8400 50  0000 L CNN
-F 2 "Capacitor_SMD:C_0805_2012Metric" H 8200 8500 50  0001 C CNN
-F 3 "" H 8200 8500 50  0001 C CNN
-	1    8200 8500
-	1    0    0    -1
-$EndComp
-Wire Wire Line
-	8200 8400 8200 8250
-Wire Wire Line
-	8200 8600 8200 8900
-Wire Wire Line
-	8200 8900 7650 8900
-Wire Wire Line
-	7650 8900 7650 8850
-Wire Wire Line
-	7650 8900 7650 9000
-Connection ~ 7650 8900
-Text Label 8350 8250 0    50   ~ 0
-3V3+
-Wire Wire Line
-	7950 8250 8200 8250
-Connection ~ 8200 8250
-Wire Wire Line
-	8200 8250 8350 8250
-Text Label 8850 8550 0    50   ~ 0
-3V3+
-$Comp
-L Diode:1N4148W D7
-U 1 1 5BF6DCC5
-P 8850 8700
-F 0 "D7" V 8896 8620 50  0000 R CNN
-F 1 "1N4148W" V 8805 8620 50  0000 R CNN
-F 2 "Diode_SMD:D_SOD-323" H 8850 8525 50  0001 C CNN
-F 3 "https://www.vishay.com/docs/85748/1n4148w.pdf" H 8850 8700 50  0001 C CNN
-	1    8850 8700
-	0    -1   -1   0
-$EndComp
-Wire Notes Line
-	8050 8700 8750 8700
-Text Notes 8300 8700 0    50   ~ 0
-As close \nas possible
 Text Label 8850 8900 0    50   ~ 0
 3V3_RTC
@@
 Wire Wire Line
 	1400 7350 1500 7350
-Text Notes 8200 8150 0    50   ~ 0
-3.3V + Vf(D6)
 Wire Wire Line
 	2150 1150 2650 1150
@@
 Wire Wire Line
 	3150 1600 3150 1700
+$Comp
+L Device:Q_NMOS_GSD Q6
+U 1 1 5BEDB255
+P 8400 8500
+F 0 "Q6" V 8743 8500 50  0000 C CNN
+F 1 "AO3401" V 8652 8500 50  0000 C CNN
+F 2 "Package_TO_SOT_SMD:SOT-23" H 8600 8600 50  0001 C CNN
+F 3 "~" H 8400 8500 50  0001 C CNN
+	1    8400 8500
+	0    1    -1   0
+$EndComp
+Wire Wire Line
+	8600 8400 8850 8400
+Wire Wire Line
+	8850 8400 8850 8650
+$Comp
+L power:+3V3 #PWR032
+U 1 1 5BEF0D30
+P 8100 8350
+F 0 "#PWR032" H 8100 8200 50  0001 C CNN
+F 1 "+3V3" H 8115 8523 50  0000 C CNN
+F 2 "" H 8100 8350 50  0001 C CNN
+F 3 "" H 8100 8350 50  0001 C CNN
+	1    8100 8350
+	1    0    0    -1
+$EndComp
+Wire Wire Line
+	8100 8350 8100 8400
+Wire Wire Line
+	8100 8400 8150 8400
+$Comp
+L ntp_7seg_clock-rescue:Q_NPN_BEC-device Q5
+U 1 1 5BEFBA07
+P 7600 8900
+F 0 "Q5" H 7790 8946 50  0000 L CNN
+F 1 "Q_NPN_BEC" H 7790 8855 50  0000 L CNN
+F 2 "Package_TO_SOT_SMD:SOT-23" H 7791 8809 50  0001 L CNN
+F 3 "" H 7600 8900 50  0000 C CNN
+	1    7600 8900
+	1    0    0    -1
+$EndComp
+Wire Wire Line
+	8400 8700 8150 8700
+$Comp
+L power:GND #PWR031
+U 1 1 5BF1BD39
+P 7700 9100
+F 0 "#PWR031" H 7700 8850 50  0001 C CNN
+F 1 "GND" H 7705 8927 50  0000 C CNN
+F 2 "" H 7700 9100 50  0000 C CNN
+F 3 "" H 7700 9100 50  0000 C CNN
+	1    7700 9100
+	1    0    0    -1
+$EndComp
+$Comp
+L ntp_7seg_clock-rescue:R-device R15
+U 1 1 5BF270CC
+P 7250 8900
+F 0 "R15" V 7250 8850 50  0000 L CNN
+F 1 "10k" V 7350 8800 50  0000 L CNN
+F 2 "Resistor_SMD:R_0603_1608Metric" V 7180 8900 50  0001 C CNN
+F 3 "" H 7250 8900 50  0000 C CNN
+	1    7250 8900
+	0    -1   -1   0
+$EndComp
+$Comp
+L power:+3V3 #PWR019
+U 1 1 5BF2737D
+P 6950 8900
+F 0 "#PWR019" H 6950 8750 50  0001 C CNN
+F 1 "+3V3" H 6965 9073 50  0000 C CNN
+F 2 "" H 6950 8900 50  0001 C CNN
+F 3 "" H 6950 8900 50  0001 C CNN
+	1    6950 8900
+	1    0    0    -1
+$EndComp
+Wire Wire Line
+	7100 8900 6950 8900
+$Comp
+L ntp_7seg_clock-rescue:R-device R16
+U 1 1 5BEC997B
+P 8150 8550
+F 0 "R16" V 8150 8500 50  0000 L CNN
+F 1 "10k" V 8250 8450 50  0000 L CNN
+F 2 "Resistor_SMD:R_0603_1608Metric" V 8080 8550 50  0001 C CNN
+F 3 "" H 8150 8550 50  0000 C CNN
+	1    8150 8550
+	1    0    0    -1
+$EndComp
+Connection ~ 8150 8400
+Wire Wire Line
+	8150 8400 8200 8400
+Connection ~ 8150 8700
+Wire Wire Line
+	8150 8700 7700 8700
 $EndSCHEMATC

Commit message: Layout fix
Connections:
- wire segments 194 -> 195
Changed lines of the file:
@@
 Wire Wire Line
 	8150 8700 7700 8700
+$Comp
+L power:GND #PWR?
+U 1 1 5BF5A579
+P 1400 1350
+F 0 "#PWR?" H 1400 1100 50  0001 C CNN
+F 1 "GND" H 1405 1177 50  0000 C CNN
+F 2 "" H 1400 1350 50  0001 C CNN
+F 3 "" H 1400 1350 50  0001 C CNN
+	1    1400 1350
+	1    0    0    -1
+$EndComp
+Wire Wire Line
+	1150 1350 1400 1350
 $EndSCHEMATC
